Commit message: feat(ag95): define gripper TCP frame

File: src/dh_gripper/dh_gripper_ros-master/dh_robotics_ag95_gripper/dh_robotics_ag95_description/urdf/dh_robotics_ag95_gripper.urdf.xacro (robot description, xacro)
@@ -27,4 +27,13 @@
             </inertial>
         </link>
+        <!-- Task TCP at the nominal AG95 grasp center.
+             +Z points from gripper base toward the fingers.
+             Initial measured offset: 175 mm. -->
+        <link name="${prefix}ag95_tcp"/>
+        <joint name="${prefix}ag95_tcp_joint" type="fixed">
+            <parent link="${prefix}gripper_base_link"/>
+            <child link="${prefix}ag95_tcp"/>
+            <origin xyz="0 0 0.175" rpy="0 0 0"/>
+        </joint>
         <gazebo reference="${prefix}gripper_base_link">
             <implicitSpringDamper>1</implicitSpringDamper>
